Commit message: Small fixes and improvements in branch

File: puzzlebot_description/urdf/xacros/gazebo_plugins.xacro (robot description, xacro)
@@ -2,5 +2,4 @@
 <robot xmlns:xacro="http://www.ros.org/wiki/xacro" name="puzzlebot">
     <xacro:property name="update_rate" value="60" />
-    <xacro:property name="namespace" value="puzzlebot" />
     <!-- Includes the differential drive controller and joint state publisher -->
     <xacro:macro name="diff_drive_controller">
@@ -10,7 +9,4 @@
                 <!-- Update rate in Hertz -->
                 <update_rate>${update_rate}</update_rate>
-                <ros>
-                    <namespace>${namespace}</namespace>
-                </ros>
                 <!-- wheels -->
                 <left_joint>wheel_left_joint</left_joint>
@@ -40,5 +36,4 @@
             <plugin name="joint_state_publisher" filename="libgazebo_ros_joint_state_publisher.so">
                 <ros>
-                    <namespace>${namespace}</namespace>
                     <remapping>~/out:=joint_states</remapping>
                 </ros>
@@ -84,7 +79,4 @@
                 </camera>
                 <plugin name="rgb_camera_plugin" filename="libgazebo_ros_camera.so">
-                    <ros>
-                        <namespace>${namespace}</namespace>
-                    </ros>
                     <camera_name>camera</camera_name>
                     <frame_name>camera_frame</frame_name>
@@ -118,5 +110,4 @@
                 <plugin name="laser" filename="libgazebo_ros_ray_sensor.so">
                     <ros>
-                        <namespace>${namespace}</namespace>
                         <remapping>~/out:=scan</remapping>
                     </ros>
