Commit message: Small fixes and improvements

File: ros_gz_puzzlebot_description/urdf/puzzlebot.urdf.xacro (robot description, xacro)
@@ -1,8 +1,8 @@
 <?xml version="1.0"?>
 <robot xmlns:xacro="http://www.ros.org/wiki/xacro" name="puzzlebot">
-    <xacro:include filename="$(find puzzlebot_description)/urdf/xacros/chassis.xacro" />
-    <xacro:include filename="$(find puzzlebot_description)/urdf/xacros/gazebo_plugins.xacro" />
-    <xacro:include filename="$(find puzzlebot_description)/urdf/xacros/geometric_primitives.xacro" />
-    <xacro:include filename="$(find puzzlebot_description)/urdf/xacros/wheels.xacro" />
+    <xacro:include filename="$(find ros_gz_puzzlebot_description)/urdf/xacros/chassis.xacro" />
+    <xacro:include filename="$(find ros_gz_puzzlebot_description)/urdf/xacros/gazebo_plugins.xacro" />
+    <xacro:include filename="$(find ros_gz_puzzlebot_description)/urdf/xacros/geometric_primitives.xacro" />
+    <xacro:include filename="$(find ros_gz_puzzlebot_description)/urdf/xacros/wheels.xacro" />
     <!-- Get the current puzzlebot model -->
     <xacro:arg name="model" default="$(env PUZZLEBOT_MODEL)" />

File: ros_gz_puzzlebot_description/urdf/xacros/chassis.xacro (robot description, xacro)
@@ -26,5 +26,5 @@
             <xacro:inertial_box width="${width}" depth="${depth}" height="${height}" z="${z_offset}"
                 mass="${mass}" />
-            <xacro:mesh filename="package://puzzlebot_description/meshes/chassis/${mesh}" />
+            <xacro:mesh filename="package://ros_gz_puzzlebot_description/meshes/chassis/${mesh}" />
         </link>
     </xacro:macro>
@@ -40,5 +40,5 @@
         <link name="camera_link">
             <xacro:mesh
-                filename="package://puzzlebot_description/meshes/camera.dae"
+                filename="package://ros_gz_puzzlebot_description/meshes/camera.dae"
                 R="${R}" P="${P}" Y="${Y}" />
             <xacro:collision_box width="${width}" depth="${depth}" height="${height}"
@@ -61,5 +61,5 @@
         <link name="lidar_link">
             <xacro:mesh
-                filename="package://puzzlebot_description/meshes/lidar.dae"
+                filename="package://ros_gz_puzzlebot_description/meshes/lidar.dae"
                 R="${R}" P="${P}" Y="${Y}" />
             <xacro:collision_box width="${width}" depth="${depth}" height="${height}"

File: ros_gz_puzzlebot_description/urdf/xacros/gazebo_plugins.xacro (robot description, xacro)
@@ -2,15 +2,11 @@
 <robot xmlns:xacro="http://www.ros.org/wiki/xacro" name="puzzlebot">
     <xacro:property name="update_rate" value="60" />
-    <xacro:property name="namespace" value="puzzlebot" />
     <!-- Includes the differential drive controller and joint state publisher -->
     <xacro:macro name="diff_drive_controller">
         <!-- Differential Drive Controller -->
         <gazebo>
-            <plugin name="differential_drive_controller" filename="libgazebo_ros_diff_drive.so">
+            <plugin name="gz::sim::systems::DiffDrive" filename="gz-sim-diff-drive-system">
                 <!-- Update rate in Hertz -->
-                <update_rate>${update_rate}</update_rate>
-                <ros>
-                    <namespace>${namespace}</namespace>
-                </ros>
+                <odom_publisher_frequency>${update_rate}</odom_publisher_frequency>
                 <!-- wheels -->
                 <left_joint>wheel_left_joint</left_joint>
@@ -18,31 +14,20 @@
                 <!-- kinematics -->
                 <wheel_separation>0.179</wheel_separation>
-                <wheel_diameter>0.09334</wheel_diameter>
+                <wheel_radius>${0.09334/2}</wheel_radius>
                 <!-- limits -->
-                <max_wheel_acceleration>1.0</max_wheel_acceleration>
-                <max_wheel_torque>1.0</max_wheel_torque>
+                <max_linear_acceleration>1.0</max_linear_acceleration>
                 <!-- input -->
-                <command_topic>cmd_vel</command_topic>
+                <topic>cmd_vel</topic>
                 <!-- output -->
-                <publish_odom>true</publish_odom>
-                <publish_odom_tf>true</publish_odom_tf>
-                <publish_wheel_tr>false</publish_wheel_tr>
-                <publish_wheel_joint_state>false</publish_wheel_joint_state>
-                <odometry_source>0</odometry_source>
-                <odometry_topic>odom</odometry_topic>
-                <odometry_frame>odom</odometry_frame>
-                <robot_base_frame>base_link</robot_base_frame>
-                <legacy_mode>false</legacy_mode>
+                <odom_topic>odom</odom_topic>
+                <frame_id>odom</frame_id>
+                <child_frame_id>base_link</child_frame_id>
+                <tf_topic>/tf</tf_topic>
             </plugin>
         </gazebo>
         <!-- Joint State Publisher Plugin -->
         <gazebo>
-            <plugin name="joint_state_publisher" filename="libgazebo_ros_joint_state_publisher.so">
-                <ros>
-                    <namespace>${namespace}</namespace>
-                    <remapping>~/out:=joint_states</remapping>
-                </ros>
-                <!-- Update rate in Hertz -->
-                <update_rate>${update_rate}</update_rate>
+            <plugin name="gz::sim::systems::JointStatePublisher" filename="gz-sim-joint-state-publisher-system">
+                <topic>joint_states</topic>
                 <joint_name>wheel_right_joint</joint_name>
                 <joint_name>wheel_left_joint</joint_name>
@@ -57,7 +42,10 @@
         <gazebo reference="camera_frame">
             <sensor name="rgb_camera" type="camera">
+                <always_on>true</always_on>
+                <topic>camera/image_raw</topic>
+                <visualize>true</visualize>
                 <update_rate>${update_rate}</update_rate>  <!-- Camera frame rate (Hz) -->
                 <camera name="rgb_camera">
-                    <always_on>true</always_on>
+                    <camera_info_topic>camera/camera_info</camera_info_topic>
                     <horizontal_fov>1.3962634</horizontal_fov>
                     <image>
@@ -83,11 +71,4 @@
                     </noise>
                 </camera>
-                <plugin name="rgb_camera_plugin" filename="libgazebo_ros_camera.so">
-                    <ros>
-                        <namespace>${namespace}</namespace>
-                    </ros>
-                    <camera_name>camera</camera_name>
-                    <frame_name>camera_frame</frame_name>
-                </plugin>
             </sensor>
         </gazebo>
@@ -96,13 +77,15 @@
     <xacro:macro name="lidar_plugin">
         <gazebo reference="lidar_frame">
-            <sensor name="lidar_sensor" type="ray">
+            <sensor name="lidar_sensor" type="gpu_lidar">
                 <pose>0 0 0 0 0 0</pose>
-                <visualize>false</visualize>
-                <update_rate>${update_rate}</update_rate>
+                <visualize>true</visualize>
+                <update_rate>10</update_rate>
                 <always_on>true</always_on>
-                <ray>
+                <topic>scan</topic>
+                <gz_frame_id>lidar_frame</gz_frame_id>
+                <lidar>
                     <scan>
                         <horizontal>
-                            <samples>200</samples>
+                            <samples>360</samples>
                             <resolution>1.0</resolution>
                             <min_angle>-3.14</min_angle>
@@ -111,16 +94,9 @@
                     </scan>
                     <range>
-                        <min>0.045</min>
-                        <max>5.0</max>
-                        <resolution>0.01</resolution>
+                        <min>0.15</min>
+                        <max>8.0</max>
+                        <resolution>0.1</resolution>
                     </range>
-                </ray>
-                <plugin name="laser" filename="libgazebo_ros_ray_sensor.so">
-                    <ros>
-                        <namespace>${namespace}</namespace>
-                        <remapping>~/out:=scan</remapping>
-                    </ros>
-                    <output_type>sensor_msgs/LaserScan</output_type>
-                </plugin>
+                </lidar>
             </sensor>
         </gazebo>

File: ros_gz_puzzlebot_description/urdf/xacros/wheels.xacro (robot description, xacro)
@@ -9,5 +9,5 @@
         <link name="${link_name}">
             <xacro:mesh
-                filename="package://puzzlebot_description/meshes/wheel.dae"
+                filename="package://ros_gz_puzzlebot_description/meshes/wheel.dae"
                 R="${R}" P="${P}" Y="${Y}" />
             <xacro:collision_cylinder radius="${radius}" length="${length}" R="${R}" P="${P}"
@@ -32,5 +32,5 @@
         <link name="caster_wheel_support">
             <xacro:mesh
-                filename="package://puzzlebot_description/meshes/caster_wheel_support.dae"
+                filename="package://ros_gz_puzzlebot_description/meshes/caster_wheel_support.dae"
             />
             <xacro:collision_box width="${width}" depth="${depth}" height="${height}"

Commit message: Update: Puzzlebot description includes now a forklift that can be included using the environment variable INCLUDE_FORKLIFT

File: ros_gz_puzzlebot_description/urdf/puzzlebot.urdf.xacro (robot description, xacro)
@@ -5,6 +5,8 @@
     <xacro:include filename="$(find ros_gz_puzzlebot_description)/urdf/xacros/geometric_primitives.xacro" />
     <xacro:include filename="$(find ros_gz_puzzlebot_description)/urdf/xacros/wheels.xacro" />
+    <xacro:include filename="$(find ros_gz_puzzlebot_description)/urdf/xacros/forklift.xacro"/>
     <!-- Get the current puzzlebot model -->
     <xacro:arg name="model" default="$(env PUZZLEBOT_MODEL)" />
+    <xacro:arg name="include_forklift" default="$(env INCLUDE_FORKLIFT)" />
     <!-- Chassis -->
     <link name="base_link" />
@@ -51,3 +53,13 @@
         <xacro:lidar_plugin />
     </xacro:if>
+    <xacro:if value="${'$(arg include_forklift)' == 'true'}">
+        <!-- Forklift (if required) -->
+        <xacro:forklift />
+        <xacro:fixed_joint parent="chassis_link" child="forklift_base" x="0.105" z="0.027123"/>
+    </xacro:if>
+    <gazebo reference="base_link">
+        <keyword>
+            <allow_auto_disable>false</allow_auto_disable>
+        </keyword>
+    </gazebo>
 </robot>

File: ros_gz_puzzlebot_description/urdf/xacros/wheels.xacro (robot description, xacro)
@@ -46,5 +46,5 @@
             <axis xyz="0 0 1" />
             <origin xyz="0 0 -0.0165" rpy="0 0 0" />
-            <limit effort="1000.0" velocity="100.0" />
+            <limit effort="1000000.0" velocity="100.0" />
             <dynamics damping="0.0" friction="0.1" />
         </joint>
